File: kelly/isolator-pcb/isolator.kicad_pcb (KiCad board)
At the start: 2 copper layers, 50 x 32 mm, 19 parts

Commit message: Route GND1 straight into U1 pin 4
The run to pin 4 dropped to y=16.8, went east, then turned back up -- margin
against crossing the pin-2/3 signal stubs that was never needed, since those
sit at y=12.365 and 13.635 and pin 4 is at 14.905, already below both.

Go straight in: down x=19.5, east at y=14.905. Three segments become two.
Clearances measured on the result: 0.45 mm from the vertical to the via
annuli, 0.77 mm from the run-in to the pin-3 stub, 0.62 mm to VIA_VIB. DRC
0 violations / 0 unconnected.

Side effect worth noting: C2's return to pin 4 goes 10.3 mm -> 7.2 mm, which
retires the "longer than ideal for a bypass cap" caveat the old comment
carried.

Does not touch where the C2 spur runs, which is the change that was reverted.

Co-Authored-By: Claude Opus 5 <noreply@anthropic.com>
Claude-Session: https://claude.ai/code/session_01UdkbaD5XWcGgk61KsSv1pw
Routing:
- net GND1: track 47.1 -> 44.0 mm
Changed lines of the file:
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@@
 (segment (start 112.040 61.500) (end 119.500 61.500) (width 0.5) (layer "F.Cu") (net 2))
 (segment (start 119.500 61.500) (end 119.500 60.540) (width 0.5) (layer "F.Cu") (net 2))
-(segment (start 119.500 61.500) (end 119.500 66.800) (width 0.5) (layer "F.Cu") (net 2))
-(segment (start 119.500 66.800) (end 121.400 66.800) (width 0.5) (layer "F.Cu") (net 2))
-(segment (start 121.400 66.800) (end 122.300 64.905) (width 0.5) (layer "F.Cu") (net 2))
+(segment (start 119.500 61.500) (end 119.500 64.905) (width 0.5) (layer "F.Cu") (net 2))
+(segment (start 119.500 64.905) (end 122.300 64.905) (width 0.5) (layer "F.Cu") (net 2))
 (segment (start 114.580 59.500) (end 114.580 55.500) (width 0.6) (layer "F.Cu") (net 1))
 (segment (start 105.500 63.000) (end 118.300 62.365) (width 0.5) (layer "B.Cu") (net 5))
